File: board/board.kicad_pcb (KiCad board)
At the start: 2 copper layers, 21 x 13 mm, 1 part

Commit message: imported legacy version
Parts:
- removed LOGO1: Logo_Open_Hardware_Small, Symbol:OSHW-Symbol_6.7x6mm_SilkScreen
- added C1: 100nF, Capacitor_SMD:C_0805_2012Metric, F.Cu at (90.0, 94.5)
- added C2: 1uF, Capacitor_SMD:C_0805_2012Metric, F.Cu at (84.0, 83.0)
- added C3: 1uF, Capacitor_SMD:C_0805_2012Metric, F.Cu at (95.5, 94.0)
- added C4: 100uF, Capacitor_SMD:CP_Elec_8x5.4, F.Cu at (112.5, 98.5)
- added J1: 001_I2C, on_edge:on_edge_2x05_device, F.Cu at (77.0, 80.0)
- added J2: 003_power, on_edge:on_edge_2x05_device, F.Cu at (77.0, 96.5)
- added J3: Conn_01x06_Male, Connector_PinHeader_2.54mm:PinHeader_1x06_P2.54mm_Vertical, F.Cu at (112.5, 78.0)
- added Q1: FDMC86102LZ, AI-footprints:TRANS_FDMC86102LZ, F.Cu at (114.4, 84.0)
- added Q2: FDMC86102LZ, AI-footprints:TRANS_FDMC86102LZ, F.Cu at (109.5, 84.0)
- added Q3: FDMC86102LZ, AI-footprints:TRANS_FDMC86102LZ, F.Cu at (104.7, 84.0)
- added Q4: FDMC86102LZ, AI-footprints:TRANS_FDMC86102LZ, F.Cu at (100.1, 83.9)
- added R1: 2.2k, Resistor_SMD:R_0402_1005Metric, F.Cu at (91.9, 83.2)
- added R2: 250m, Resistor_SMD:R_2512_6332Metric, F.Cu at (109.5, 89.9)
- added R3: 250m, Resistor_SMD:R_2512_6332Metric, F.Cu at (104.6, 89.9)
- added R4: 250m, Resistor_SMD:R_2512_6332Metric, F.Cu at (114.4, 89.9)
- added R5: 250m, Resistor_SMD:R_2512_6332Metric, F.Cu at (100.0, 89.9)
- added R6: 0R, Resistor_SMD:R_0402_1005Metric, F.Cu at (97.2, 81.2)
- added TP1: int_tp, TestPoint:TestPoint_Pad_2.0x2.0mm, F.Cu at (88.2, 79.0)
- added TP10: tp, TestPoint:TestPoint_Pad_2.0x2.0mm, F.Cu at (91.2, 79.0)
- added TP11: tp, TestPoint:TestPoint_Pad_2.0x2.0mm, F.Cu at (94.2, 79.0)
- added TP12: tp, TestPoint:TestPoint_Pad_2.0x2.0mm, F.Cu at (97.2, 79.0)
- added TP2: tp, TestPoint:TestPoint_Pad_2.0x2.0mm, F.Cu at (84.5, 99.5)
- added TP3: tp, TestPoint:TestPoint_Pad_2.0x2.0mm, F.Cu at (87.5, 99.5)
- added TP4: tp, TestPoint:TestPoint_Pad_2.0x2.0mm, F.Cu at (90.5, 99.5)
- added TP5: tp, TestPoint:TestPoint_Pad_2.0x2.0mm, F.Cu at (93.5, 99.5)
- added TP6: tp, TestPoint:TestPoint_Pad_2.0x2.0mm, F.Cu at (96.5, 99.5)
- added TP7: tp, TestPoint:TestPoint_Pad_2.0x2.0mm, F.Cu at (99.5, 99.5)
- added TP8: tp, TestPoint:TestPoint_Pad_2.0x2.0mm, F.Cu at (102.5, 99.5)
- added TP9: tp, TestPoint:TestPoint_Pad_2.0x2.0mm, F.Cu at (105.5, 99.5)
- added U3: LTC4266AIUHF-4#PBF, Package_DFN_QFN:QFN-38-1EP_5x7mm_P0.5mm_EP3.15x5.15mm, F.Cu at (92.4, 88.4)
Routing:
- net GND: track 0.00 -> 135.5 mm, vias 0 -> 15
- net /Controller/poe+: track 0.00 -> 58.8 mm
- net +3V3: track 0.00 -> 43.9 mm, vias 0 -> 3
- net /Controller/SW4: track 0.00 -> 32.2 mm
- net Net-(Q1-Pad3): track 0.00 -> 30.3 mm
- net /Controller/SW3: track 0.00 -> 26.1 mm
- net Net-(J1-Pad10): track 0.00 -> 25.0 mm, vias 0 -> 2
- net Net-(Q1-Pad1): track 0.00 -> 24.8 mm
- net Net-(Q2-Pad3): track 0.00 -> 23.1 mm
- net /Controller/SW2: track 0.00 -> 22.2 mm
- net Net-(Q2-Pad1): track 0.00 -> 19.5 mm
- net Net-(TP9-Pad1): track 0.00 -> 17.8 mm
- net /Controller/SDA: track 0.00 -> 16.3 mm, vias 0 -> 2
- net /Controller/SW1: track 0.00 -> 16.1 mm
- net Net-(TP8-Pad1): track 0.00 -> 15.6 mm
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- added copper zone on B.Cu, net GND
- added copper zone on F.Cu, net GND
Other:
- board size 21 x 13 mm -> 41 x 29 mm
- rule pad_to_mask_clearance: 0 -> 0.04
- board text added: "osf.001.v0.2"
- board text added: "osf.003.v0.2"
- board text added: "osf.b029.v0.1"
