File: board/board.kicad_sch (KiCad schematic)
At the start: 1 part

Commit message: imported legacy version
Parts:
- removed LOGO1: Logo_Open_Hardware_Small, Symbol:OSHW-Symbol_6.7x6mm_SilkScreen, symbol Graphic:Logo_Open_Hardware_Small
- added J1: (no value), symbol board-rescue:001_I2C-put_on_edge
- added J2: (no value), symbol board-rescue:003_power-put_on_edge
- added J3: (no value), symbol Connector:Conn_01x06_Male
- added TP1: (no value), symbol Connector:TestPoint
Connections:
- new net: J1.10 (5V), J2.10 (5V)
- new net +3V3: J1.9 (3.3V), J2.9 (3.3V)
- new net Controller/SCL: J1.3 (SCL)
- new net Controller/SDA: J1.2 (SDA)
- new net Controller/SW1: J3.4 (Pin_4)
- new net Controller/SW2: J3.3 (Pin_3)
- new net Controller/SW3: J3.2 (Pin_2)
- new net Controller/SW4: J3.1 (Pin_1)
- new net Controller/int: TP1.1
- new net Controller/poe+: J3.5 (Pin_5)
- new net GND: J1.1 (GND), J2.1 (GND), J2.2 (GND), J2.3 (GND), J2.4 (GND), J2.5 (GND), J3.6 (Pin_6)
- no-connect marks 0 -> 6
Other:
- removed sheet implementation
- added sheet Controller (Controller.kicad_sch)
- note removed: "Input connectors go here"
- note removed: "Output connectors go here"
